Commit message: Added Tiller Design Changes

File: deweeder_ws_ros/install/deweeder_robot/share/deweeder_robot/urdf/deweeder_robot.urdf (robot description, URDF)
Before this commit: robot tracked_deweeder, 8 links, 7 joints
Links:
- added link tiller_link, mass 0.8; collision box size=0.35 0.08 0.02; visual box size=0.35 0.08 0.02
Joints:
- added joint tiller_joint: type fixed, parent base_chassis, child tiller_link, origin xyz=0.28 0 0.02 rpy=0.2 0 0

File: deweeder_ws_ros/src/deweeder_robot/urdf/deweeder_robot.urdf (robot description, URDF)
Before this commit: robot tracked_deweeder, 8 links, 7 joints
Links:
- added link tiller_link, mass 0.8; collision box size=0.35 0.08 0.02; visual box size=0.35 0.08 0.02
Joints:
- added joint tiller_joint: type fixed, parent base_chassis, child tiller_link, origin xyz=0.28 0 0.02 rpy=0.2 0 0
