Commit message: Completing the remaining infra

File: src/weedbot_simulation_tertill/urdf/weedbot.urdf (robot description, URDF)
Before this commit: robot weedbot, 5 links, 4 joints
Links:
- added link belly_sensor_link, mass 0.01; collision cylinder length=0.005 radius=0.08; visual cylinder length=0.005 radius=0.08
- added link bumper_front_link, mass 0.01; collision box size=0.01 0.22 0.08; visual box size=0.01 0.22 0.08
Joints:
- added joint belly_sensor_joint: type fixed, parent base_link, child belly_sensor_link, origin xyz=0 0 -0.015
- added joint bumper_front_joint: type fixed, parent base_link, child bumper_front_link, origin xyz=0.110 0 0.06
